Commit message: Mapping and Localization added

File: mobi_description/urdf/gazebo.xacro (robot description, xacro)
@@ -98,5 +98,5 @@
         </sensor>
     </gazebo>
-    <gazebo reference="lidar_link">
+    <gazebo reference="laser_link">
         <sensor name="lidar" type="gpu_lidar">
             <pose>0 0 0 0 0 0</pose>
@@ -105,5 +105,5 @@
             <topic>scan</topic>
             <update_rate>5</update_rate>
-            <gz_frame_id>lidar_link</gz_frame_id>
+            <gz_frame_id>laser_link</gz_frame_id>
             <lidar>
                 <scan>

File: mobi_description/urdf/mobi_base.xacro (robot description, xacro)
@@ -131,5 +131,5 @@
     <child link="right_castor_wheel"/>
 </joint>
-<link name="lidar_link">
+<link name="laser_link">
     <inertial>
         <origin xyz="-0.154 0.0 -0.19" rpy="0.0 0.0 0.0"/>
@@ -151,8 +151,8 @@
     </collision>
 </link>
-<joint name="lidar_joint" type="fixed">
+<joint name="laser_joint" type="fixed">
     <origin xyz="0.154 0.0 0.19" rpy="0.0 0.0 0.0"/>
     <parent link="base_link"/>
-    <child link="lidar_link"/>
+    <child link="laser_link"/>
 </joint>
 <link name="camera_link">
